Commit message: gripper not working well now

File: catkin_ws/src/ocs2_robotic_assets/resources/mobile_manipulator/ridgeback_ur5/urdf/ridgeback_ur5_robotiq.urdf (robot description, URDF)
Before this commit: robot ridgeback, 38 links, 37 joints
Links:
- link axle_link: geometry visual mesh filename=package://ocs2_robotic_assets/resources/mobile_manipulator/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
- link chassis_link: geometry collision mesh filename=package://ocs2_robotic_assets/resources/mobile_manipulator/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; visual mesh filename=package://ocs2_robotic_assets/resources/mobile_manipulator/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
- link front_cover_link: geometry visual mesh filename=package://ocs2_robotic_assets/resources/mobile_manipulator/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
- link front_left_wheel_link: geometry collision cylinder length=0.079 radius=0.0759; visual mesh filename=package://ocs2_robotic_assets/resources/mobile_manipulator/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
- link front_lights_link: geometry visual mesh filename=package://ocs2_robotic_assets/resources/mobile_manipulator/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
- link front_right_wheel_link: geometry collision cylinder length=0.079 radius=0.0759; visual mesh filename=package://ocs2_robotic_assets/resources/mobile_manipulator/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
- link front_rocker_link: geometry visual mesh filename=package://ocs2_robotic_assets/resources/mobile_manipulator/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
- link left_inner_finger: geometry collision mesh filename=package://ocs2_robotic_assets/resources/mobile_manipulator/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; visual mesh filename=package://ocs2_robotic_assets/resources/mobile_manipulator/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
- link left_inner_knuckle: geometry collision mesh filename=package://ocs2_robotic_assets/resources/mobile_manipulator/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; visual mesh filename=package://ocs2_robotic_assets/resources/mobile_manipulator/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
- link left_outer_finger: geometry collision mesh filename=package://ocs2_robotic_assets/resources/mobile_manipulator/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; visual mesh filename=package://ocs2_robotic_assets/resources/mobile_manipulator/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
- link left_outer_knuckle: geometry collision mesh filename=package://ocs2_robotic_assets/resources/mobile_manipulator/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; visual mesh filename=package://ocs2_robotic_assets/resources/mobile_manipulator/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
- link left_side_cover_link: geometry visual mesh filename=package://ocs2_robotic_assets/resources/mobile_manipulator/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
- link rear_cover_link: geometry visual mesh filename=package://ocs2_robotic_assets/resources/mobile_manipulator/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
- link rear_left_wheel_link: geometry collision cylinder length=0.079 radius=0.0759; visual mesh filename=package://ocs2_robotic_assets/resources/mobile_manipulator/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
- link rear_lights_link: geometry visual mesh filename=package://ocs2_robotic_assets/resources/mobile_manipulator/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
- link rear_right_wheel_link: geometry collision cylinder length=0.079 radius=0.0759; visual mesh filename=package://ocs2_robotic_assets/resources/mobile_manipulator/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
- link rear_rocker_link: geometry visual mesh filename=package://ocs2_robotic_assets/resources/mobile_manipulator/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
- link right_inner_finger: geometry collision mesh filename=package://ocs2_robotic_assets/resources/mobile_manipulator/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; visual mesh filename=package://ocs2_robotic_assets/resources/mobile_manipulator/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
- link right_inner_knuckle: geometry collision mesh filename=package://ocs2_robotic_assets/resources/mobile_manipulator/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; visual mesh filename=package://ocs2_robotic_assets/resources/mobile_manipulator/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
- link right_outer_finger: geometry collision mesh filename=package://ocs2_robotic_assets/resources/mobile_manipulator/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; visual mesh filename=package://ocs2_robotic_assets/resources/mobile_manipulator/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
- link right_outer_knuckle: geometry collision mesh filename=package://ocs2_robotic_assets/resources/mobile_manipulator/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; visual mesh filename=package://ocs2_robotic_assets/resources/mobile_manipulator/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
- link right_side_cover_link: geometry visual mesh filename=package://ocs2_robotic_assets/resources/mobile_manipulator/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
- link robotiq_85_base_link: geometry collision mesh filename=package://ocs2_robotic_assets/resources/mobile_manipulator/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; visual mesh filename=package://ocs2_robotic_assets/resources/mobile_manipulator/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
- link top_link: geometry collision mesh filename=package://ocs2_robotic_assets/resources/mobile_manipulator/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; visual mesh filename=package://ocs2_robotic_assets/resources/mobile_manipulator/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
- link ur_arm_base_link_inertia: geometry collision mesh filename=package://ocs2_robotic_assets/resources/mobile_manipulator/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; visual mesh filename=package://ocs2_robotic_assets/resources/mobile_manipulator/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
- link ur_arm_forearm_link: geometry collision mesh filename=package://ocs2_robotic_assets/resources/mobile_manipulator/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; visual mesh filename=package://ocs2_robotic_assets/resources/mobile_manipulator/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
- link ur_arm_shoulder_link: geometry collision mesh filename=package://ocs2_robotic_assets/resources/mobile_manipulator/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; visual mesh filename=package://ocs2_robotic_assets/resources/mobile_manipulator/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
- link ur_arm_upper_arm_link: geometry collision mesh filename=package://ocs2_robotic_assets/resources/mobile_manipulator/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; visual mesh filename=package://ocs2_robotic_assets/resources/mobile_manipulator/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
- link ur_arm_wrist_1_link: geometry collision mesh filename=package://ocs2_robotic_assets/resources/mobile_manipulator/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; visual mesh filename=package://ocs2_robotic_assets/resources/mobile_manipulator/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
- link ur_arm_wrist_2_link: geometry collision mesh filename=package://ocs2_robotic_assets/resources/mobile_manipulator/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; visual mesh filename=package://ocs2_robotic_assets/resources/mobile_manipulator/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
- link ur_arm_wrist_3_link: geometry collision mesh filename=package://ocs2_robotic_assets/resources/mobile_manipulator/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; visual mesh filename=package://ocs2_robotic_assets/resources/mobile_manipulator/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
