Commit message: working on prismatic gripper

File: edf_env/robot/ridgeback_ur5/ridgeback_ur5_robotiq_debug.urdf (robot description, URDF)
Before this commit: robot ridgeback, 42 links, 41 joints
Links:
- removed link left_finger_z_fake
- removed link right_finger_z_fake
- removed link right_inner_finger_fake
- added link finger_z_fake; visual box size=0.1 0.01 0.05
- link left_inner_finger_fake: geometry visual mesh filename=meshes/robotiq/inner_finger_fine.stl
Joints:
- removed joint left_finger_z_joint_fake
- removed joint right_finger_z_joint_fake
- removed joint right_inner_finger_joint_fake
- added joint finger_z_joint_fake: type prismatic, parent robotiq_85_base_link, child finger_z_fake, origin xyz=0 0 0.07 rpy=0 0 0, axis 0 0 1, limit lower=-1 upper=1 effort=1000 velocity=2.0
- joint left_inner_finger_joint: child left_inner_finger_fake -> left_inner_finger
- joint left_inner_finger_joint_fake: child left_inner_finger -> left_inner_finger_fake; parent left_finger_z_fake -> finger_z_fake
- joint right_inner_finger_joint: child right_inner_finger_fake -> right_inner_finger; mimic (none) -> joint=finger_joint multiplier=1 offset=0
