Commit message: fixed atan2

File: edf_env/robot/ridgeback_ur5/ridgeback_ur5_robotiq.urdf (robot description, URDF)
Before this commit: robot ridgeback, 42 links, 41 joints
Joints:
- joint left_finger_z_joint_fake: origin xyz=0 0 0.07 rpy=0 0 0 -> xyz=0 0 0. rpy=0 0 0
- joint left_inner_finger_joint_fake: origin xyz=0.014 0 0 rpy=0 0 0 -> xyz=0 0 0 rpy=0 0 0
- joint right_finger_z_joint_fake: origin xyz=0 0 0.07 rpy=0 0 0 -> xyz=0 0 0. rpy=0 0 0
- joint right_inner_finger_joint_fake: origin xyz=-0.014 0 0 rpy=0 0 0 -> xyz=0 0 0 rpy=0 0 0
