Commit message: simplify mesh train0, test1, test2

File: edf_env/assets/mug_task/mugs/test/mug3/mug.urdf (robot description, URDF)
Before this commit: robot mug, 1 links, 0 joints
Links:
- link base_link: geometry collision mesh filename=mug.obj scale=0.05 0.05 0.05; visual mesh filename=mug.obj scale=0.05 0.05 0.05

File: edf_env/assets/mug_task/mugs/test/mug4/mug.urdf (robot description, URDF)
Before this commit: robot mug, 1 links, 0 joints
Links:
- link base_link: geometry collision mesh filename=mug.obj scale=0.015 0.015 0.015; visual mesh filename=mug.obj scale=0.015 0.015 0.015

File: edf_env/assets/mug_task/mugs/test/mug5/mug.urdf (robot description, URDF)
Before this commit: robot mug, 1 links, 0 joints
Links:
- link base_link: geometry collision mesh filename=mug.dae scale=0.03 0.03 0.03; visual mesh filename=mug.dae scale=0.03 0.03 0.03

File: edf_env/assets/mug_task/mugs/train/mug0/_mug.urdf (robot description, URDF)
Before this commit: robot mug, 1 links, 0 joints
Links:
- link base_link: geometry collision mesh filename=mug.obj; visual mesh filename=mug.obj
