Commit message: simplified meshes

File: edf_env/assets/mug_task/mugs/test/mug10/mug.urdf (robot description, URDF)
Before this commit: robot coffee_cup_sharp.urdf, 1 links, 0 joints
Links:
- removed link baseLink
- added link base_link, mass 0.1; collision mesh filename=mug_simplified.stl scale=1 1 1; visual mesh filename=mug_simplified.stl scale=1 1 1

File: edf_env/assets/mug_task/mugs/test/mug3/mug.urdf (robot description, URDF)
Before this commit: robot mug, 1 links, 0 joints
Links:
- link base_link: mass 1 -> 0.1; geometry collision mesh filename=mug_simplified.stl scale=1 1 1; visual mesh filename=mug_simplified.stl scale=1 1 1

File: edf_env/assets/mug_task/mugs/test/mug4/mug.urdf (robot description, URDF)
Before this commit: robot mug, 1 links, 0 joints
Links:
- link base_link: mass 1 -> 0.1; geometry collision mesh filename=mug_simplified.stl scale=1 1 1; visual mesh filename=mug_simplified.stl scale=1 1 1

File: edf_env/assets/mug_task/mugs/test/mug5/mug.urdf (robot description, URDF)
Before this commit: robot mug, 1 links, 0 joints
Links:
- link base_link: mass 1 -> 0.1; geometry collision mesh filename=mug_simplified.stl scale=1 1 1; visual mesh filename=mug_simplified.stl scale=1 1 1

File: edf_env/assets/mug_task/mugs/test/mug6/mug.urdf (robot description, URDF)
Before this commit: robot mug.urdf, 1 links, 0 joints
Links:
- removed link baseLink
- added link base_link, mass 0.1; collision mesh filename=mug_simplified.stl scale=1 1 1; visual mesh filename=mug_simplified.stl scale=1 1 1

File: edf_env/assets/mug_task/mugs/test/mug7/mug.urdf (robot description, URDF)
Before this commit: robot tea_cup.urdf, 1 links, 0 joints
Links:
- removed link baseLink
- added link base_link, mass 0.1; collision mesh filename=mug_simplified.stl scale=1 1 1; visual mesh filename=mug_simplified.stl scale=1 1 1

File: edf_env/assets/mug_task/mugs/test/mug8/mug.urdf (robot description, URDF)
Before this commit: robot widecup.urdf, 1 links, 0 joints
Links:
- removed link baseLink
- added link base_link, mass 0.1; collision mesh filename=mug_simplified.stl scale=1 1 1; visual mesh filename=mug_simplified.stl scale=1 1 1

File: edf_env/assets/mug_task/mugs/test/mug9/mug.urdf (robot description, URDF)
Before this commit: robot coffee_cup_sharp.urdf, 1 links, 0 joints
Links:
- removed link baseLink
- added link base_link, mass 0.1; collision mesh filename=mug_simplified.stl scale=1 1 1; visual mesh filename=mug_simplified.stl scale=1 1 1
